Commit message: Add files via upload

File: AutoBot/urdf/AutoBot.urdf (robot description, URDF)
Before this commit: robot AutoBot, 17 links, 16 joints
Joints:
- joint base_link_to_center_camera: origin xyz=0.58 0 0.5 rpy=0 0 0 -> xyz=0.58 0 1.2 rpy=0 0.3 0

Commit message: Add files via upload

File: AutoBot/urdf/AutoBot.urdf (robot description, URDF)
Before this commit: robot AutoBot, 17 links, 16 joints
Joints:
- joint base_link_to_center_camera: origin xyz=0.58 0 1.2 rpy=0 0.3 0 -> xyz=0.58 0 0.5 rpy=0 0 0

Commit message: Add files via upload

File: AutoBot/urdf/AutoBot.urdf (robot description, URDF)
Before this commit: robot AutoBot, 17 links, 16 joints
Joints:
- joint base_link_to_center_camera: origin xyz=0.58 0 0.5 rpy=0 0 0 -> xyz=1.5 0 1.5 rpy=0 1.6 0

Commit message: Add files via upload

File: AutoBot/urdf/AutoBot.urdf (robot description, URDF)
Before this commit: robot AutoBot, 17 links, 16 joints
Joints:
- joint base_link_to_kinect_cam: origin xyz=0.55 0 0.8 rpy=0 0.2617 0 -> xyz=0.55 0 0.8 rpy=0 0.5 0
